File: PCB/mcu.kicad_sch (KiCad schematic)
At the start: 39 parts, among them J201 switch, J202 switch, U201 W25Q128JVSIQ, U202 RP2040, Y201 12MHz

Commit message: Update net labels
Parts:
- gave numbers to parts that had none: 12
- renumbered C201 to C101, C202 to C102, C208 to C103, C203 to C104, C207 to C105, C209 to C106, C210 to C107, C211 to C108, C212 to C109, C213 to C110, C214 to C111, C204 to C112, C205 to C113, C206 to C114, J201 to J101, J202 to J102, R207 to R101, R206 to R102, R201 to R103, R203 to R104, R204 to R105, R205 to R106, U201 to U101, U202 to U102, Y201 to Y101
Connections:
- net VDD is gone; now on net +3V3: U102.1 (IOVDD), U102.10 (IOVDD), U102.22 (IOVDD), U102.33 (IOVDD), U102.42 (IOVDD), U102.43 (ADC_AVDD), U102.44 (VREG_IN), U102.48 (USB_VDD), U102.49 (IOVDD)
- net +3.3V: no longer C116.1, L101.2, R110.1, U103.6 (VOS)
- net +3V3: now also C116.1, L101.2, R110.1, U103.6 (VOS)
- net XIN: now also U102.20 (XIN)
- net XOUT: now also U102.21 (XOUT)
Other:
- note added: "Make sure C114 is close to pin 45 of RP2040"
- note added: "Make sure C3 is close to pin 44 of RP2040"
- note added: "Make sure R5 and R6 are close to RP2040"
- note added: "Make sure U4 is close to J3"
- note removed: "Make sure C6 is close to pin 45 of RP2040"
- note removed: "Make sure C8 is close to pin 44 of RP2040"
- note removed: "Make sure R4 and R5 are close to RP2040"
- note removed: "Make sure U2 is close to J1"
