File: PCB/mcu.kicad_sch (KiCad schematic)
At the start: 39 parts, among them J101 switch, J102 switch, J103 USB4510-03-1-A, J104 CONN_DISPLAY, U101 W25Q128JVSIQ, U102 RP2040, U103 TPS62172DSG, U104 USBLC6-2SC6, Y101 12MHz

Commit message: Left side 'done'
Connections:
- net COL-1: now also U102.31 (GPIO20); no longer U102.7 (GPIO5)
- net COL-2: now also U102.32 (GPIO21); no longer U102.8 (GPIO6)
- net COL-3: now also U102.34 (GPIO22); no longer U102.9 (GPIO7)
- net COL-4: now also U102.35 (GPIO23); no longer U102.11 (GPIO8)
- net COL-5: now also U102.36 (GPIO24); no longer U102.12 (GPIO9)
- net ROW-1: now also U102.39 (GPIO27_ADC1); no longer U102.32 (GPIO21)
- net ROW-2: now also U102.38 (GPIO26_ADC0); no longer U102.31 (GPIO20)
- no-connect marks 20 -> 13
Changed lines of the file:
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@@
   (no_connect (at 156.21 72.39))
   (no_connect (at 83.82 129.54))
-  (no_connect (at 156.21 138.43))
   (no_connect (at 218.44 44.45))
   (no_connect (at 156.21 102.87))
@@
   (no_connect (at 156.21 95.25))
   (no_connect (at 156.21 87.63))
-  (no_connect (at 156.21 123.19))
   (no_connect (at 156.21 92.71))
-  (no_connect (at 156.21 135.89))
   (no_connect (at 156.21 90.17))
-  (no_connect (at 156.21 130.81))
   (no_connect (at 83.82 127))
   (no_connect (at 156.21 69.85))
   (no_connect (at 156.21 67.31))
   (no_connect (at 259.08 31.75))
-  (no_connect (at 156.21 120.65))
-  (no_connect (at 156.21 133.35))
-  (no_connect (at 156.21 118.11))
   (wire (pts (xy 156.21 102.87) (xy 152.4 102.87))
     (stroke (width 0) (type default) (color 0 0 0 0))
@@
     (stroke (width 0) (type default) (color 0 0 0 0))
   )
-  (wire (pts (xy 158.75 82.55) (xy 152.4 82.55))
-    (stroke (width 0) (type default) (color 0 0 0 0))
-  )
   (wire (pts (xy 226.06 160.02) (xy 226.06 163.83))
     (stroke (width 0) (type default) (color 0 0 0 0))
@@
     (stroke (width 0) (type default) (color 0 0 0 0))
   )
-  (wire (pts (xy 152.4 115.57) (xy 158.75 115.57))
-    (stroke (width 0) (type default) (color 0 0 0 0))
-  )
   (wire (pts (xy 157.48 54.61) (xy 157.48 57.15))
     (stroke (width 0) (type default) (color 0 0 0 0))
   )
-  (wire (pts (xy 158.75 80.01) (xy 152.4 80.01))
-    (stroke (width 0) (type default) (color 0 0 0 0))
-  )
   (wire (pts (xy 270.51 46.99) (xy 270.51 53.34))
     (stroke (width 0) (type default) (color 0 0 0 0))
@@
     (stroke (width 0) (type default) (color 0 0 0 0))
   )
+  (wire (pts (xy 158.75 123.19) (xy 152.4 123.19))
+    (stroke (width 0) (type default) (color 0 0 0 0))
+  )
   (wire (pts (xy 102.87 39.37) (xy 100.33 39.37))
     (stroke (width 0) (type default) (color 0 0 0 0))
@@
     (stroke (width 0) (type default) (color 0 0 0 0))
   )
+  (wire (pts (xy 158.75 120.65) (xy 152.4 120.65))
+    (stroke (width 0) (type default) (color 0 0 0 0))
+  )
   (wire (pts (xy 152.4 87.63) (xy 156.21 87.63))
     (stroke (width 0) (type default) (color 0 0 0 0))
   )
-  (wire (pts (xy 156.21 123.19) (xy 152.4 123.19))
-    (stroke (width 0) (type default) (color 0 0 0 0))
-  )
   (wire (pts (xy 203.2 116.84) (xy 212.09 116.84))
     (stroke (width 0) (type default) (color 0 0 0 0))
@@
     (stroke (width 0) (type default) (color 0 0 0 0))
   )
-  (wire (pts (xy 156.21 120.65) (xy 152.4 120.65))
-    (stroke (width 0) (type default) (color 0 0 0 0))
-  )
   (wire (pts (xy 133.35 44.45) (xy 133.35 39.37))
     (stroke (width 0) (type default) (color 0 0 0 0))
@@
     (stroke (width 0) (type default) (color 0 0 0 0))
   )
-  (wire (pts (xy 152.4 135.89) (xy 156.21 135.89))
-    (stroke (width 0) (type default) (color 0 0 0 0))
-  )
   (wire (pts (xy 162.56 100.33) (xy 152.4 100.33))
     (stroke (width 0) (type default) (color 0 0 0 0))
@@
     (stroke (width 0) (type default) (color 0 0 0 0))
   )
+  (wire (pts (xy 152.4 133.35) (xy 158.75 133.35))
+    (stroke (width 0) (type default) (color 0 0 0 0))
+  )
   (wire (pts (xy 152.4 107.95) (xy 158.75 107.95))
     (stroke (width 0) (type default) (color 0 0 0 0))
@@
     (stroke (width 0) (type default) (color 0 0 0 0))
   )
+  (wire (pts (xy 158.75 113.03) (xy 152.4 113.03))
+    (stroke (width 0) (type default) (color 0 0 0 0))
+  )
   (wire (pts (xy 236.22 154.94) (xy 252.73 154.94))
     (stroke (width 0) (type default) (color 0 0 0 0))
   )
-  (wire (pts (xy 152.4 130.81) (xy 156.21 130.81))
-    (stroke (width 0) (type default) (color 0 0 0 0))
-  )
   (wire (pts (xy 156.21 90.17) (xy 152.4 90.17))
     (stroke (width 0) (type default) (color 0 0 0 0))
@@
     (stroke (width 0) (type default) (color 0 0 0 0))
   )
-  (wire (pts (xy 152.4 133.35) (xy 156.21 133.35))
-    (stroke (width 0) (type default) (color 0 0 0 0))
-  )
   (wire (pts (xy 257.81 128.27) (xy 257.81 127))
     (stroke (width 0) (type default) (color 0 0 0 0))
@@
     (stroke (width 0) (type default) (color 0 0 0 0))
   )
-  (wire (pts (xy 158.75 85.09) (xy 152.4 85.09))
-    (stroke (width 0) (type default) (color 0 0 0 0))
-  )
   (wire (pts (xy 226.06 163.83) (xy 236.22 163.83))
     (stroke (width 0) (type default) (color 0 0 0 0))
@@
     (stroke (width 0) (type default) (color 0 0 0 0))
   )
+  (wire (pts (xy 158.75 115.57) (xy 152.4 115.57))
+    (stroke (width 0) (type default) (color 0 0 0 0))
+  )
   (wire (pts (xy 269.24 116.84) (xy 269.24 119.38))
     (stroke (width 0) (type default) (color 0 0 0 0))
@@
     (stroke (width 0) (type default) (color 0 0 0 0))
   )
-  (wire (pts (xy 152.4 138.43) (xy 156.21 138.43))
-    (stroke (width 0) (type default) (color 0 0 0 0))
-  )
   (wire (pts (xy 233.68 152.4) (xy 252.73 152.4))
     (stroke (width 0) (type default) (color 0 0 0 0))
@@
     (stroke (width 0) (type default) (color 0 0 0 0))
   )
-  (wire (pts (xy 158.75 74.93) (xy 152.4 74.93))
-    (stroke (width 0) (type default) (color 0 0 0 0))
-  )
   (wire (pts (xy 152.4 67.31) (xy 156.21 67.31))
     (stroke (width 0) (type default) (color 0 0 0 0))
@@
     (stroke (width 0) (type default) (color 0 0 0 0))
   )
-  (wire (pts (xy 156.21 118.11) (xy 152.4 118.11))
-    (stroke (width 0) (type default) (color 0 0 0 0))
-  )
   (wire (pts (xy 255.27 119.38) (xy 255.27 116.84))
     (stroke (width 0) (type default) (color 0 0 0 0))
@@
     (stroke (width 0) (type default) (color 0 0 0 0))
   )
+  (wire (pts (xy 152.4 130.81) (xy 158.75 130.81))
+    (stroke (width 0) (type default) (color 0 0 0 0))
+  )
   (wire (pts (xy 248.92 124.46) (xy 248.92 130.81))
     (stroke (width 0) (type default) (color 0 0 0 0))
@@
     (stroke (width 0) (type default) (color 0 0 0 0))
   )
+  (wire (pts (xy 158.75 118.11) (xy 152.4 118.11))
+    (stroke (width 0) (type default) (color 0 0 0 0))
+  )
   (wire (pts (xy 95.25 187.96) (xy 95.25 189.23))
     (stroke (width 0) (type default) (color 0 0 0 0))
@@
     (stroke (width 0) (type default) (color 0 0 0 0))
   )
-  (wire (pts (xy 158.75 77.47) (xy 152.4 77.47))
-    (stroke (width 0) (type default) (color 0 0 0 0))
-  )
   (wire (pts (xy 76.2 97.79) (xy 88.9 97.79))
     (stroke (width 0) (type default) (color 0 0 0 0))
@@
   )
   (wire (pts (xy 100.33 39.37) (xy 100.33 44.45))
-    (stroke (width 0) (type default) (color 0 0 0 0))
-  )
-  (wire (pts (xy 152.4 113.03) (xy 158.75 113.03))
     (stroke (width 0) (type default) (color 0 0 0 0))
   )
@@
     (effects (font (size 1.27 1.27)) (justify left bottom))
   )
-  (hierarchical_label "COL-1" (shape input) (at 158.75 74.93 0)
+  (hierarchical_label "COL-1" (shape input) (at 158.75 113.03 0)
+    (effects (font (size 1.27 1.27)) (justify left))
+  )
+  (hierarchical_label "COL-4" (shape input) (at 158.75 120.65 0)
     (effects (font (size 1.27 1.27)) (justify left))
   )
@@
     (effects (font (size 1.27 1.27)) (justify left))
   )
-  (hierarchical_label "COL-2" (shape input) (at 158.75 77.47 0)
+  (hierarchical_label "ROW-1" (shape input) (at 158.75 133.35 0)
     (effects (font (size 1.27 1.27)) (justify left))
   )
@@
     (effects (font (size 1.27 1.27)) (justify left))
   )
-  (hierarchical_label "COL-4" (shape input) (at 158.75 82.55 0)
-    (effects (font (size 1.27 1.27)) (justify left))
-  )
-  (hierarchical_label "COL-5" (shape input) (at 158.75 85.09 0)
-    (effects (font (size 1.27 1.27)) (justify left))
-  )
-  (hierarchical_label "COL-3" (shape input) (at 158.75 80.01 0)
+  (hierarchical_label "COL-3" (shape input) (at 158.75 118.11 0)
+    (effects (font (size 1.27 1.27)) (justify left))
+  )
+  (hierarchical_label "COL-2" (shape input) (at 158.75 115.57 0)
+    (effects (font (size 1.27 1.27)) (justify left))
+  )
+  (hierarchical_label "ROW-2" (shape input) (at 158.75 130.81 0)
     (effects (font (size 1.27 1.27)) (justify left))
   )
@@
     (effects (font (size 1.27 1.27)) (justify left))
   )
-  (hierarchical_label "ROW-1" (shape input) (at 158.75 115.57 0)
-    (effects (font (size 1.27 1.27)) (justify left))
-  )
-  (hierarchical_label "ROW-2" (shape input) (at 158.75 113.03 0)
-    (effects (font (size 1.27 1.27)) (justify left))
-  )
+  (hierarchical_label "COL-5" (shape input) (at 158.75 123.19 0)
+    (effects (font (size 1.27 1.27)) (justify left))
+  )

Commit message: Right ride
Connections:
- net COL-1: now also U102.29 (GPIO18); no longer U102.31 (GPIO20)
- net COL-2: now also U102.30 (GPIO19); no longer U102.32 (GPIO21)
- net COL-3: now also U102.31 (GPIO20); no longer U102.34 (GPIO22)
- net ROW-1: now also U102.14 (GPIO11); no longer U102.39 (GPIO27_ADC1)
- net ROW-2: now also U102.13 (GPIO10); no longer U102.38 (GPIO26_ADC0)
- net ROW-3: now also U102.12 (GPIO9); no longer U102.30 (GPIO19)
- net ROW-4: now also U102.11 (GPIO8); no longer U102.29 (GPIO18)
- no-connect marks 13 -> 20
