File: PCB/mcu.kicad_sch (KiCad schematic)
At the start: 39 parts, among them J101 switch, J102 switch, J103 USB4510-03-1-A, J104 CONN_DISPLAY, U101 W25Q128JVSIQ, U102 RP2040, U103 TPS62172DSG, U104 USBLC6-2SC6, Y101 12MHz

Commit message: fix errors
Changed lines of the file:
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@@
   (junction (at 212.09 127) (diameter 0) (color 0 0 0 0)
   )
-  (junction (at 264.16 116.84) (diameter 0) (color 0 0 0 0)
-  )
   (junction (at 50.8 129.54) (diameter 0) (color 0 0 0 0)
   )
@@
   )
   (junction (at 102.87 39.37) (diameter 0) (color 0 0 0 0)
-  )
-  (junction (at 243.84 160.02) (diameter 0) (color 0 0 0 0)
   )
   (no_connect (at 156.21 74.93))
@@
     (stroke (width 0) (type default) (color 0 0 0 0))
   )
-  (wire (pts (xy 257.81 116.84) (xy 264.16 116.84))
-    (stroke (width 0) (type default) (color 0 0 0 0))
-  )
   (wire (pts (xy 83.82 127) (xy 88.9 127))
     (stroke (width 0) (type default) (color 0 0 0 0))
@@
     (stroke (width 0) (type default) (color 0 0 0 0))
   )
-  (wire (pts (xy 264.16 114.3) (xy 264.16 116.84))
-    (stroke (width 0) (type default) (color 0 0 0 0))
-  )
   (wire (pts (xy 213.36 31.75) (xy 213.36 34.29))
     (stroke (width 0) (type default) (color 0 0 0 0))
@@
     (stroke (width 0) (type default) (color 0 0 0 0))
   )
-  (wire (pts (xy 264.16 116.84) (xy 269.24 116.84))
+  (wire (pts (xy 257.81 116.84) (xy 269.24 116.84))
     (stroke (width 0) (type default) (color 0 0 0 0))
   )
@@
   )
   (wire (pts (xy 212.09 125.73) (xy 212.09 127))
-    (stroke (width 0) (type default) (color 0 0 0 0))
-  )
-  (wire (pts (xy 243.84 160.02) (xy 241.3 160.02))
     (stroke (width 0) (type default) (color 0 0 0 0))
   )
@@
     (pin "6")
   )
-  (symbol (lib_id "power:PWR_FLAG") (at 241.3 160.02 180) (unit 1)
-    (in_bom yes) (on_board yes)
-    (property "Reference" "#FLG0201" (id 0) (at 241.3 161.925 0)
-      (effects (font (size 1.27 1.27)) hide)
-    )
-    (property "Value" "PWR_FLAG" (id 1) (at 241.3 163.83 0))
-    (property "Footprint" "" (id 2) (at 241.3 160.02 0)
-      (effects (font (size 1.27 1.27)) hide)
-    )
-    (property "Datasheet" "~" (id 3) (at 241.3 160.02 0)
-      (effects (font (size 1.27 1.27)) hide)
-    )
-    (pin "1")
-  )
   (symbol (lib_id "Device:C") (at 49.53 60.96 90) (unit 1)
     (in_bom yes) (on_board yes)
@@
     (pin "2")
   )
-  (symbol (lib_id "power:PWR_FLAG") (at 264.16 114.3 0) (unit 1)
-    (in_bom yes) (on_board yes)
-    (property "Reference" "#FLG0102" (id 0) (at 264.16 112.395 0)
-      (effects (font (size 1.27 1.27)) hide)
-    )
-    (property "Value" "PWR_FLAG" (id 1) (at 264.16 110.49 0))
-    (property "Footprint" "" (id 2) (at 264.16 114.3 0)
-      (effects (font (size 1.27 1.27)) hide)
-    )
-    (property "Datasheet" "~" (id 3) (at 264.16 114.3 0)
-      (effects (font (size 1.27 1.27)) hide)
-    )
-    (pin "1")
-  )
   (symbol (lib_id "Device:R") (at 217.17 156.21 180) (unit 1)
