File: PCB/keyboard.kicad_pcb (KiCad board)
At the start: 2 copper layers, 125.5 x 102.1 mm, 154 parts, among them J101 switch, J102 switch, J103 USB4510-03-1-A, J104 CONN_DISPLAY, J105 AudioJack4, J201 switch, J202 switch, J203 USB4510-03-1-A, J204 CONN_DISPLAY, J205 AudioJack4, U101 W25Q128JVSIQ, U102 RP2040, U103 TPS62172DSG, U104 USBLC6-2SC6, U105 USBLC6-2SC6, U201 W25Q128JVSIQ, U202 RP2040, U203 TPS62172DSG, U204 USBLC6-2SC6, U205 USBLC6-2SC6, Y101 12MHz, Y201 12MHz

Commit message: Work
Parts:
- moved J104 58.7 mm to (139.6, 57.6)
- moved D120 53.8 mm to (149.1, 30.8)
- moved D119 28.8 mm to (152.6, 30.8)
- moved C102 28.7 mm to (145.3, 44.3)
- moved U101 28.6 mm to (148.9, 48.4)
- moved J102 28.0 mm to (134.5, 88.2)
- moved C111 27.9 mm to (146.8, 57.5)
- moved C108 27.9 mm to (135.2, 53.8)
- moved R104 27.9 mm to (142.6, 63.4)
- moved R106 27.9 mm to (139.6, 50.1)
- moved C101 27.9 mm to (144.7, 64.6)
- moved C104 27.9 mm to (142.7, 64.6)
- moved C113 27.9 mm to (139.3, 63.0)
- moved Y101 27.9 mm to (143.8, 67.3)
- moved C103 27.9 mm to (137.5, 51.1)
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Connections:
- D116 pad 1: /Left Matix/ROW-4 -> /Left MCU/ROW-4
- D117 pad 1: /Left Matix/ROW-4 -> /Left MCU/ROW-4
- D118 pad 1: /Left Matix/ROW-4 -> /Left MCU/ROW-4
- U102 pad 13: /Left MCU/COL-6 -> unconnected-(U102-Pad13)
- U102 pad 29: unconnected-(U102-Pad29) -> /Left MCU/ROW-4
- U102 pad 30: unconnected-(U102-Pad30) -> /Left MCU/ROW-3
- U102 pad 31: unconnected-(U102-Pad31) -> /Left MCU/ROW-2
- U102 pad 32: unconnected-(U102-Pad32) -> /Left MCU/ROW-1
- U102 pad 4: /Left MCU/ROW-1 -> unconnected-(U102-Pad4)
- U102 pad 5: /Left MCU/ROW-2 -> unconnected-(U102-Pad5)
- U102 pad 6: /Left MCU/ROW-3 -> unconnected-(U102-Pad6)
- U202 pad 13: /Right MCU/COL-6 -> unconnected-(U202-Pad13)
- U202 pad 29: unconnected-(U202-Pad29) -> /Right MCU/ROW-4
- U202 pad 30: unconnected-(U202-Pad30) -> /Right MCU/ROW-3
- U202 pad 31: unconnected-(U202-Pad31) -> /Right MCU/ROW-2
- U202 pad 32: unconnected-(U202-Pad32) -> /Right MCU/ROW-1
- U202 pad 4: /Right MCU/ROW-1 -> unconnected-(U202-Pad4)
- U202 pad 5: /Right MCU/ROW-2 -> unconnected-(U202-Pad5)
- U202 pad 6: /Right MCU/ROW-3 -> unconnected-(U202-Pad6)
Routing:
- net /Left MCU/COL-5: track 0.00 -> 136.6 mm, vias 0 -> 5
- net /Left MCU/ROW-3: track 0.00 -> 130.0 mm
- net /Left MCU/ROW-1: track 0.00 -> 124.3 mm
- net /Left MCU/ROW-2: track 0.00 -> 114.2 mm
- net /Left MCU/COL-3: track 0.00 -> 98.6 mm, vias 0 -> 4
- net /Left MCU/COL-4: track 0.00 -> 97.9 mm, vias 0 -> 4
- net /Left MCU/ROW-4: track 0.00 -> 70.0 mm
- net /Left MCU/COL-2: track 0.00 -> 52.5 mm, vias 0 -> 3
- net /Left MCU/COL-1: track 6.77 -> 46.8 mm
- net /Left MCU/USB_D-: track 34.7 -> 6.61 mm
- net /Left MCU/USB_D+: track 34.7 -> 6.61 mm
- net Net-(D118-Pad2): track 0.00 -> 27.6 mm
- net /Left MCU/SDA: track 3.19 -> 27.1 mm
- net VBUS: track 37.7 -> 13.9 mm, vias 4 -> 2
- net /Left MCU/SCL: track 3.79 -> 22.4 mm
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Other:
- board size 125.5 x 102.1 mm -> 129.9 x 102.1 mm

Commit message: Add mounting holes
Parts:
- added H101: MountingHole_Pad, Footprints:M2_HOLE_v3, F.Cu at (45.6, 49.0)
- added H102: MountingHole_Pad, Footprints:M2_HOLE_v3, F.Cu at (102.6, 49.0)
- added H103: MountingHole_Pad, Footprints:M2_HOLE_v3, F.Cu at (45.6, 89.4)
- added H104: MountingHole_Pad, Footprints:M2_HOLE_v3, F.Cu at (102.6, 89.4)
- added H105: MountingHole_Pad, Footprints:M2_HOLE_v3, F.Cu at (142.3, 94.1)
- added H201: MountingHole_Pad, Footprints:M2_HOLE_v3, F.Cu at (871.1, 99.3)
- added H202: MountingHole_Pad, Footprints:M2_HOLE_v3, F.Cu at (859.5, 105.6)
- added H203: MountingHole_Pad, Footprints:M2_HOLE_v3, F.Cu at (859.5, 99.7)
- added H204: MountingHole_Pad, Footprints:M2_HOLE_v3, F.Cu at (865.5, 105.6)
- added H205: MountingHole_Pad, Footprints:M2_HOLE_v3, F.Cu at (865.5, 99.7)
- moved D116 6.40 mm to (102.0, 100.5)
- moved D110 1.97 mm to (100.0, 44.2)
Routing:
- net /Left MCU/ROW-1: track 124.3 -> 130.8 mm
- net Net-(D116-Pad2): track 15.7 -> 20.5 mm
- net /Left MCU/ROW-3: track 130.0 -> 127.5 mm
- net /Left MCU/ROW-4: track 70.0 -> 71.9 mm
- net Net-(D110-Pad2): track 15.7 -> 14.5 mm
- net /Left MCU/COL-5: track 136.6 -> 137.2 mm
- net /Left MCU/COL-2: track 52.5 -> 53.1 mm

Commit message: Metric
Parts:
- moved R108 108.6 mm to (250.0, 68.7), turned to 90 degrees
- moved J105 108.6 mm to (263.3, 76.5)
- moved C101 108.4 mm to (253.0, 62.2), turned to 90 degrees
- moved MX118 108.1 mm to (243.8, 107.0)
- moved MX117 108.0 mm to (222.3, 100.0)
- moved D116 108.0 mm to (209.8, 94.0)
- moved D117 108.0 mm to (232.3, 94.0)
- moved U105 107.9 mm to (258.0, 72.7)
- moved MX104 107.9 mm to (162.8, 36.0)
- moved MX105 107.9 mm to (162.8, 55.0)
- moved MX106 107.9 mm to (162.8, 74.0)
- moved MX111 107.9 mm to (200.8, 55.0)
- moved MX110 107.9 mm to (200.8, 36.0)
- moved MX112 107.9 mm to (200.8, 74.0)
- moved MX115 107.9 mm to (219.8, 74.0)
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Connections:
- J104 pad 2: +3.3V -> +3V3
- J204 pad 2: +3.3V -> +3V3
- Y101 pad 4: +3.3V -> +3V3
- Y201 pad 4: +3.3V -> +3V3
Routing:
- net /Left MCU/COL-1: track 46.8 -> 147.5 mm, vias 0 -> 2
- net /Left MCU/COL-2: track 53.1 -> 136.2 mm, vias 3 -> 4
- net /Left MCU/COL-3: track 98.6 -> 157.2 mm, vias 4 -> 5
- net /Left MCU/COL-4: track 97.9 -> 132.7 mm, vias 4 -> 5
- net /Left MCU/TX: track 0.00 -> 32.5 mm
- net /Left MCU/RX: track 0.00 -> 27.3 mm
- net /Left MCU/COL-5: track 137.2 -> 119.5 mm
- net /Left MCU/ROW-1: track 130.8 -> 118.7 mm
- net +3V3: track 34.8 -> 44.5 mm, vias 2 -> 6
- net /Left MCU/SCL: track 22.4 -> 31.3 mm, vias 0 -> 2
- net /Left MCU/SDA: track 27.1 -> 34.3 mm, vias 0 -> 2
- net Net-(D116-Pad2): track 20.5 -> 15.2 mm
- net VBUS: track 13.9 -> 18.7 mm, vias 2 -> 3
- net /Left MCU/~{RESET}: track 0.00 -> 3.60 mm
- net /Left MCU/XIN: track 12.8 -> 9.98 mm, vias 2 -> 0
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Other:
- board size 129.9 x 102.1 mm -> 131 x 103 mm

Commit message: Add switch footprint
Parts:
- J101, J102, J201, J202: footprint Connector_PinHeader_2.54mm:PinHeader_1x02_P2.54mm_Vertical -> Footprints:SKHLACA010

Commit message: add OLED footprint
Parts:
- J104, J204: footprint Footprints:OLED_128_64 -> Footprints:SSD1306_0.96_Oled
- moved J104 18.9 mm to (259.1, 40.6)
