File: PCB/keyboard.kicad_pcb (KiCad board)
At the start: 2 copper layers, 129 x 99.1 mm, 164 parts, among them J101 switch, J102 switch, J103 USB4510-03-1-A, J104 CONN_DISPLAY, J105 AudioJack4, J201 switch, J202 switch, J203 USB4510-03-1-A, J204 CONN_DISPLAY, J205 AudioJack4, U101 W25Q128JVSIQ, U102 RP2040, U103 TPS62172DSG, U104 USBLC6-2SC6, U105 USBLC6-2SC6, U201 W25Q128JVSIQ, U202 RP2040, U203 TPS62172DSG, U204 USBLC6-2SC6, U205 USBLC6-2SC6, Y101 12MHz, Y201 12MHz

Commit message: Left side 'done'
Parts:
- moved J102 37.5 mm to (261.5, 53.2), turned to 90 degrees
- moved J101 25.4 mm to (261.5, 62.5), turned to 90 degrees
- moved J104 17.7 mm to (246.3, 55.0)
- moved D119 4.34 mm to (256.3, 29.0), turned to 90 degrees
- moved R101 4.32 mm to (256.3, 31.7), turned to 90 degrees
- moved D120 2.65 mm to (259.3, 29.0), turned to 90 degrees
- moved R102 2.14 mm to (259.3, 31.7), turned to 90 degrees
- moved C101 0.75 mm to (253.0, 63.7)
- moved Y101 0.75 mm to (250.3, 63.5)
- moved C105 0.59 mm to (239.8, 58.2)
- moved U101 0.25 mm to (253.8, 48.7)
Connections:
- J205 pad R1: (no net) -> /TRRS Connection/R_RX
- J205 pad R2: (no net) -> /TRRS Connection/R_TX
- J205 pad S: (no net) -> +3V3
- J205 pad T: (no net) -> GND
- U102 pad 11: /Left MCU/COL-4 -> unconnected-(U102-Pad11)
- U102 pad 12: /Left MCU/COL-5 -> unconnected-(U102-Pad12)
- U102 pad 31: /Left MCU/ROW-2 -> /Left MCU/COL-1
- U102 pad 32: /Left MCU/ROW-1 -> /Left MCU/COL-2
- U102 pad 34: unconnected-(U102-Pad34) -> /Left MCU/COL-3
- U102 pad 35: unconnected-(U102-Pad35) -> /Left MCU/COL-4
- U102 pad 36: unconnected-(U102-Pad36) -> /Left MCU/COL-5
- U102 pad 38: unconnected-(U102-Pad38) -> /Left MCU/ROW-2
- U102 pad 39: unconnected-(U102-Pad39) -> /Left MCU/ROW-1
- U102 pad 7: /Left MCU/COL-1 -> unconnected-(U102-Pad7)
- U102 pad 8: /Left MCU/COL-2 -> unconnected-(U102-Pad8)
- U102 pad 9: /Left MCU/COL-3 -> unconnected-(U102-Pad9)
- U105 pad 5: +3.3V -> +3V3
- U202 pad 11: /Right MCU/COL-4 -> unconnected-(U202-Pad11)
- U202 pad 12: /Right MCU/COL-5 -> unconnected-(U202-Pad12)
- U202 pad 31: /Right MCU/ROW-2 -> /Right MCU/COL-1
- U202 pad 32: /Right MCU/ROW-1 -> /Right MCU/COL-2
- U202 pad 34: unconnected-(U202-Pad34) -> /Right MCU/COL-3
- U202 pad 35: unconnected-(U202-Pad35) -> /Right MCU/COL-4
- U202 pad 36: unconnected-(U202-Pad36) -> /Right MCU/COL-5
- U202 pad 38: unconnected-(U202-Pad38) -> /Right MCU/ROW-2
- U202 pad 39: unconnected-(U202-Pad39) -> /Right MCU/ROW-1
- U202 pad 7: /Right MCU/COL-1 -> unconnected-(U202-Pad7)
- U202 pad 8: /Right MCU/COL-2 -> unconnected-(U202-Pad8)
- U202 pad 9: /Right MCU/COL-3 -> unconnected-(U202-Pad9)
Routing:
- net /Left MCU/LED: track 1.44 -> 49.5 mm, vias 1 -> 4
- net /Left MCU/~{RESET}: track 3.60 -> 38.1 mm, vias 0 -> 1
- net /Left MCU/COL-4: track 132.7 -> 154.2 mm
- net /Left MCU/COL-5: track 119.5 -> 140.7 mm
- net /Left MCU/COL-3: track 157.2 -> 178.4 mm
- net /Left MCU/COL-2: track 136.2 -> 157.2 mm
- net /Left MCU/COL-1: track 147.5 -> 168.5 mm
- net +3V3: track 44.5 -> 61.6 mm, vias 6 -> 8
- net /Left MCU/~{BOOTSEL}: track 0.00 -> 4.79 mm
- net GND: track 34.8 -> 38.8 mm, vias 27 -> 31
- net /Left MCU/ROW-2: track 111.4 -> 114.0 mm
- net /Left MCU/ROW-1: track 118.7 -> 121.3 mm
- net /Left MCU/ROW-4: track 73.6 -> 71.5 mm
- net /Left MCU/ROW-3: track 127.8 -> 125.7 mm
- net Net-(D120-Pad1): track 0.00 -> 1.45 mm
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
Commit message: More adjustments and space out trace
Parts:
- D201, D202, D203, D204, D205, D206, D207, D208, D209, D210, D211, D212, D213, D214, D215, D216, D217, D218, J203, U201, U202: moved to B.Cu
- moved J205 733.4 mm to (154.2, 95.5), turned to 90 degrees
- moved U202 705.2 mm to (171.2, 73.5), turned to 180 degrees
- moved J203 676.9 mm to (171.2, 47.0)
- moved U201 665.7 mm to (178.7, 65.5), turned to 180 degrees
- moved MX213 609.4 mm to (197.7, 52.8)
- moved MX212 590.4 mm to (216.7, 90.8)
- moved MX214 589.2 mm to (197.7, 71.8)
- moved MX215 569.1 mm to (197.7, 90.8)
- moved MX218 553.5 mm to (173.7, 123.8), turned to 25 degrees
- moved MX205 552.4 mm to (254.7, 71.8)
- moved MX209 552.0 mm to (235.7, 84.8)
- moved MX206 532.2 mm to (254.7, 90.8)
- moved MX211 530.4 mm to (216.7, 71.8)
- moved MX217 514.8 mm to (195.2, 116.8), turned to 10 degrees
- moved MX216 513.2 mm to (216.7, 114.8)
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Routing:
- net /Right MCU/QSPI_SS: track 0.00 -> 16.0 mm
- net /Right MCU/QSPI_SD1: track 0.00 -> 14.7 mm
- net GND: track 38.8 -> 51.0 mm
- net /Left MCU/ROW-1: track 121.3 -> 119.8 mm
- net /Left MCU/ROW-2: track 114.0 -> 112.9 mm
- net /Left MCU/ROW-4: track 71.5 -> 70.6 mm
- net /Left MCU/ROW-3: track 125.7 -> 124.9 mm
- net /Left MCU/COL-1: track 168.5 -> 167.8 mm
Other:
- board size 129 x 99.1 mm -> 270 x 99.1 mm
- board text added: "LEFT"

Commit message: Right ride
Parts:
- C201, C202, C203, C204, C205, C206, C207, C208, C209, C210, C211, C212, C213, C214, C215, C216, D219, D220, L201, R201, R202, R203, R204, R205, R206, R207, R208, R209, R210, R211, U203, U204, U205, Y201: moved to B.Cu
- moved C215 360.9 mm to (161.5, 49.8), turned to 180 degrees
- moved U205 359.4 mm to (159.0, 97.5), turned to -90 degrees
- moved C216 358.8 mm to (159.0, 53.0), turned to 90 degrees
- moved L201 357.0 mm to (160.7, 56.8), turned to 180 degrees
- moved R210 357.0 mm to (165.0, 54.5), turned to 90 degrees
- moved C209 328.1 mm to (165.2, 69.5), turned to 180 degrees
- moved C205 325.8 mm to (165.0, 74.5), turned to 180 degrees
- moved J201 321.9 mm to (156.2, 79.3), turned to 90 degrees
- moved C214 315.8 mm to (168.5, 67.0), turned to 90 degrees
- moved H205 315.4 mm to (168.2, 107.8)
- moved U203 315.4 mm to (161.7, 52.5), turned to -90 degrees
- moved C208 315.3 mm to (165.2, 70.8), turned to 180 degrees
- moved C212 315.3 mm to (172.7, 67.0), turned to 90 degrees
- moved R202 314.9 mm to (159.7, 46.0), turned to -90 degrees
- moved R205 314.6 mm to (170.5, 67.0), turned to -90 degrees
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Connections:
- D216 pad 1: /Right Matrix/ROW-4 -> /Right MCU/ROW-4
- D217 pad 1: /Right Matrix/ROW-4 -> /Right MCU/ROW-4
- D218 pad 1: /Right Matrix/ROW-4 -> /Right MCU/ROW-4
- J205 pad R1: /TRRS Connection/R_RX -> /TRRS Connection/R_RX_CONN
- J205 pad R2: /TRRS Connection/R_TX -> /TRRS Connection/R_TX_CONN
- U102 pad 11: unconnected-(U102-Pad11) -> /Left MCU/ROW-4
- U102 pad 12: unconnected-(U102-Pad12) -> /Left MCU/ROW-3
- U102 pad 13: unconnected-(U102-Pad13) -> /Left MCU/ROW-2
- U102 pad 14: unconnected-(U102-Pad14) -> /Left MCU/ROW-1
- U102 pad 29: /Left MCU/ROW-4 -> /Left MCU/COL-1
- U102 pad 30: /Left MCU/ROW-3 -> /Left MCU/COL-2
- U102 pad 31: /Left MCU/COL-1 -> /Left MCU/COL-3
- U102 pad 32: /Left MCU/COL-2 -> unconnected-(U102-Pad32)
- U102 pad 34: /Left MCU/COL-3 -> unconnected-(U102-Pad34)
- U102 pad 38: /Left MCU/ROW-2 -> unconnected-(U102-Pad38)
- U102 pad 39: /Left MCU/ROW-1 -> unconnected-(U102-Pad39)
- U202 pad 11: unconnected-(U202-Pad11) -> /Right MCU/ROW-4
- U202 pad 12: unconnected-(U202-Pad12) -> /Right MCU/ROW-3
- U202 pad 13: unconnected-(U202-Pad13) -> /Right MCU/ROW-2
- U202 pad 14: unconnected-(U202-Pad14) -> /Right MCU/ROW-1
- U202 pad 2: /TRRS Connection/R_TX -> /Right MCU/TX
- U202 pad 29: /Right MCU/ROW-4 -> /Right MCU/COL-1
- U202 pad 3: /TRRS Connection/R_RX -> /Right MCU/RX
- U202 pad 30: /Right MCU/ROW-3 -> /Right MCU/COL-2
- U202 pad 31: /Right MCU/COL-1 -> /Right MCU/COL-3
- U202 pad 32: /Right MCU/COL-2 -> unconnected-(U202-Pad32)
- U202 pad 34: /Right MCU/COL-3 -> unconnected-(U202-Pad34)
- U202 pad 38: /Right MCU/ROW-2 -> unconnected-(U202-Pad38)
- U202 pad 39: /Right MCU/ROW-1 -> unconnected-(U202-Pad39)
- U205 pad 1: /TRRS Connection/R_TX -> /TRRS Connection/R_TX_CONN
- U205 pad 3: /TRRS Connection/R_RX -> /TRRS Connection/R_RX_CONN
- U205 pad 4: /TRRS Connection/R_RX -> /Right MCU/RX
- U205 pad 5: +3.3V -> +3V3
- U205 pad 6: /TRRS Connection/R_TX -> /Right MCU/TX
Routing:
- net /Right MCU/COL-1: track 0.00 -> 188.2 mm, vias 0 -> 2
- net /Right MCU/COL-3: track 0.00 -> 186.1 mm, vias 0 -> 7
- net /Right MCU/COL-2: track 0.00 -> 178.1 mm, vias 0 -> 6
- net /Right MCU/COL-4: track 0.00 -> 171.6 mm, vias 0 -> 7
- net /Right MCU/ROW-1: track 0.00 -> 164.6 mm, vias 0 -> 2
- net /Right MCU/COL-5: track 0.00 -> 161.1 mm, vias 0 -> 5
- net /Right MCU/ROW-2: track 0.00 -> 118.9 mm, vias 0 -> 2
- net /Right MCU/ROW-3: track 0.00 -> 114.3 mm, vias 0 -> 2
- net +3V3: track 62.1 -> 131.5 mm, vias 8 -> 16
- net /Right MCU/ROW-4: track 0.00 -> 68.1 mm, vias 0 -> 4
- net /Right MCU/TX: track 0.00 -> 53.6 mm
- net /Right MCU/RX: track 0.00 -> 49.5 mm
- net /Right MCU/~{BOOTSEL}: track 0.00 -> 40.5 mm, vias 0 -> 4
- net /Right MCU/LED: track 0.00 -> 40.3 mm, vias 0 -> 2
- net /Right MCU/SDA: track 0.00 -> 35.7 mm, vias 0 -> 2
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- added copper zone on B.Cu, net Net-(L201-Pad1)
Other:
- outline, holes or cut-outs redrawn

Commit message: fix errors
Parts:
- added REF**: Breakaway_Tabs, Footprints:Breakaway_Tabs, F.Cu at (145.7, 40.0)
- moved J204 0.25 mm to (171.5, 71.8)
Routing:
- net Net-(D118-Pad2): track 28.1 -> 28.8 mm
Other:
- outline, holes or cut-outs redrawn

Commit message: Fix some warnings
Parts:
- removed REF**: Breakaway_Tabs, Footprints:Breakaway_Tabs
- J103, J203: value USB4510-03-1-A -> USB4510-03-1-A_GCT
Routing:
- net +3V3: track 131.7 -> 134.1 mm
- net GND: track 63.5 -> 62.4 mm
- net VBUS: track 37.8 -> 36.8 mm
- net /TRRS Connection/R_TX_CONN: track 3.38 -> 2.49 mm
- net /TRRS Connection/R_RX_CONN: track 3.31 -> 2.65 mm
- net /Right MCU/COL-4: track 171.6 -> 171.0 mm
- net Net-(C204-Pad1): track 2.84 -> 2.33 mm
Other:
- outline, holes or cut-outs redrawn
