File: PCB/keyboard.kicad_sch (KiCad schematic)
At the start: 0 parts

Commit message: Right ride
Other:
- sheet Right MCU ports: added ROW-4; removed COL-6
- sheet Right Matrix ports: added ROW-4; removed COL-6
Changed lines of the file:
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@@
+    (stroke (width 0) (type default) (color 0 0 0 0))
+  )
+  (wire (pts (xy 133.35 69.85) (xy 137.16 69.85))
     (stroke (width 0) (type default) (color 0 0 0 0))
   )
@@
     (stroke (width 0) (type default) (color 0 0 0 0))
   )
+  (wire (pts (xy 133.35 67.31) (xy 137.16 67.31))
+    (stroke (width 0) (type default) (color 0 0 0 0))
+  )
   (wire (pts (xy 133.35 58.42) (xy 137.16 58.42))
     (stroke (width 0) (type default) (color 0 0 0 0))
   )
+  (wire (pts (xy 68.58 55.88) (xy 72.39 55.88))
+    (stroke (width 0) (type default) (color 0 0 0 0))
+  )
+  (wire (pts (xy 92.71 72.39) (xy 95.25 72.39))
+    (stroke (width 0) (type default) (color 0 0 0 0))
+  )
+  (wire (pts (xy 68.58 69.85) (xy 72.39 69.85))
+    (stroke (width 0) (type default) (color 0 0 0 0))
+  )
+  (wire (pts (xy 133.35 55.88) (xy 137.16 55.88))
+    (stroke (width 0) (type default) (color 0 0 0 0))
+  )
+  (wire (pts (xy 133.35 62.23) (xy 137.16 62.23))
+    (stroke (width 0) (type default) (color 0 0 0 0))
+  )
+  (wire (pts (xy 92.71 69.85) (xy 95.25 69.85))
+    (stroke (width 0) (type default) (color 0 0 0 0))
+  )
+  (wire (pts (xy 68.58 67.31) (xy 72.39 67.31))
+    (stroke (width 0) (type default) (color 0 0 0 0))
+  )
+  (wire (pts (xy 111.76 72.39) (xy 114.3 72.39))
+    (stroke (width 0) (type default) (color 0 0 0 0))
+  )
   (wire (pts (xy 133.35 64.77) (xy 137.16 64.77))
-    (stroke (width 0) (type default) (color 0 0 0 0))
-  )
-  (wire (pts (xy 68.58 55.88) (xy 72.39 55.88))
-    (stroke (width 0) (type default) (color 0 0 0 0))
-  )
-  (wire (pts (xy 133.35 69.85) (xy 137.16 69.85))
-    (stroke (width 0) (type default) (color 0 0 0 0))
-  )
-  (wire (pts (xy 92.71 72.39) (xy 95.25 72.39))
-    (stroke (width 0) (type default) (color 0 0 0 0))
-  )
-  (wire (pts (xy 133.35 67.31) (xy 137.16 67.31))
-    (stroke (width 0) (type default) (color 0 0 0 0))
-  )
-  (wire (pts (xy 68.58 69.85) (xy 72.39 69.85))
-    (stroke (width 0) (type default) (color 0 0 0 0))
-  )
-  (wire (pts (xy 133.35 55.88) (xy 137.16 55.88))
-    (stroke (width 0) (type default) (color 0 0 0 0))
-  )
-  (wire (pts (xy 92.71 69.85) (xy 95.25 69.85))
-    (stroke (width 0) (type default) (color 0 0 0 0))
-  )
-  (wire (pts (xy 68.58 67.31) (xy 72.39 67.31))
-    (stroke (width 0) (type default) (color 0 0 0 0))
-  )
-  (wire (pts (xy 133.35 60.96) (xy 137.16 60.96))
-    (stroke (width 0) (type default) (color 0 0 0 0))
-  )
-  (wire (pts (xy 111.76 72.39) (xy 114.3 72.39))
     (stroke (width 0) (type default) (color 0 0 0 0))
   )
@@
       (effects (font (size 1.27 1.27)) (justify left top) hide)
     )
-    (pin "COL-6" input (at 133.35 60.96 0)
-      (effects (font (size 1.27 1.27)) (justify right))
-    )
     (pin "COL-3" input (at 133.35 53.34 0)
       (effects (font (size 1.27 1.27)) (justify right))
@@
       (effects (font (size 1.27 1.27)) (justify right))
     )
-    (pin "ROW-2" input (at 133.35 67.31 0)
-      (effects (font (size 1.27 1.27)) (justify right))
-    )
-    (pin "ROW-3" input (at 133.35 69.85 0)
-      (effects (font (size 1.27 1.27)) (justify right))
-    )
-    (pin "ROW-1" input (at 133.35 64.77 0)
+    (pin "ROW-2" input (at 133.35 64.77 0)
+      (effects (font (size 1.27 1.27)) (justify right))
+    )
+    (pin "ROW-3" input (at 133.35 67.31 0)
+      (effects (font (size 1.27 1.27)) (justify right))
+    )
+    (pin "ROW-1" input (at 133.35 62.23 0)
       (effects (font (size 1.27 1.27)) (justify right))
     )
@@
     (pin "TX" input (at 114.3 69.85 180)
       (effects (font (size 1.27 1.27)) (justify left))
+    )
+    (pin "ROW-4" input (at 133.35 69.85 0)
+      (effects (font (size 1.27 1.27)) (justify right))
     )
   )
@@
       (effects (font (size 1.27 1.27)) (justify left top) hide)
     )
-    (pin "ROW-2" input (at 137.16 67.31 180)
-      (effects (font (size 1.27 1.27)) (justify left))
-    )
-    (pin "ROW-3" input (at 137.16 69.85 180)
-      (effects (font (size 1.27 1.27)) (justify left))
-    )
-    (pin "ROW-1" input (at 137.16 64.77 180)
+    (pin "ROW-2" input (at 137.16 64.77 180)
+      (effects (font (size 1.27 1.27)) (justify left))
+    )
+    (pin "ROW-3" input (at 137.16 67.31 180)
+      (effects (font (size 1.27 1.27)) (justify left))
+    )
+    (pin "ROW-1" input (at 137.16 62.23 180)
       (effects (font (size 1.27 1.27)) (justify left))
     )
@@
       (effects (font (size 1.27 1.27)) (justify left))
     )
-    (pin "COL-6" input (at 137.16 60.96 180)
+    (pin "ROW-4" input (at 137.16 69.85 180)
       (effects (font (size 1.27 1.27)) (justify left))
     )
@@
       (reference "#PWR0139") (unit 1) (value "+3V3") (footprint "")
     )
+    (path "/09e2c39d-e578-4df4-966d-37f8c8def6a5/9a57038d-0c53-4b5f-bc6c-4d8d63528b5e"
+      (reference "#PWR0140") (unit 1) (value "+3V3") (footprint "")
+    )
     (path "/2be5a3e4-6545-4242-984b-805a21c5914c/37da07c0-b021-4b67-898f-f5f5ebffab8e"
       (reference "#PWR0201") (unit 1) (value "+3V3") (footprint "")
@@
       (reference "#PWR0232") (unit 1) (value "GND") (footprint "")
     )
-    (path "/09e2c39d-e578-4df4-966d-37f8c8def6a5/b0b8ef25-2a38-48ec-8397-6d64efd67bf3"
-      (reference "#PWR0233") (unit 1) (value "+3.3V") (footprint "")
-    )
     (path "/09e2c39d-e578-4df4-966d-37f8c8def6a5/db2a306d-9303-41eb-9170-d3d032aeea61"
