File: PCB/trrs_conn.kicad_sch (KiCad schematic)
At the start: 4 parts, among them J501 AudioJack4, J502 AudioJack4, U501 USBLC6-2SC6, U502 USBLC6-2SC6

Commit message: Update net labels
Parts:
- renumbered J502 to J105, J501 to J205, U502 to U105, U501 to U205
Other:
- note added: "Left TRRS"
- note added: "Right TRRS"
- moved on the sheet: J105, J205, U105, U205

Commit message: latest changes
Parts:
- U105, U205: JLCPCB (none) -> C7519
Connections:
- net L_RX: now also J105.R2, U105.1 (I/O1)
- net L_TX: now also J105.R1, U105.3 (I/O2)
- net R_RX: now also J205.R1, U205.3 (I/O2)
- net R_TX: now also J205.R2, U205.1 (I/O1)
Changed lines of the file:
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@@
     (effects (font (size 2.54 2.54)) (justify left bottom))
+  )
+  (label "R_TX" (at 53.34 120.65 0)
+    (effects (font (size 1.27 1.27)) (justify left bottom))
+  )
+  (label "L_RX" (at 52.07 63.5 0)
+    (effects (font (size 1.27 1.27)) (justify left bottom))
+  )
+  (label "L_TX" (at 52.07 60.96 0)
+    (effects (font (size 1.27 1.27)) (justify left bottom))
+  )
+  (label "R_RX" (at 53.34 118.11 0)
+    (effects (font (size 1.27 1.27)) (justify left bottom))
   )
   (hierarchical_label "R_RX" (shape input) (at 52.07 95.25 0)
@@
     )
     (property "Datasheet" "https://datasheet.lcsc.com/lcsc/1811141711_STMicroelectronics-USBLC6-2SC6_C7519.pdf" (id 3) (at 44.45 88.9 0)
+      (effects (font (size 1.27 1.27)) hide)
+    )
+    (property "JLCPCB" "C7519" (id 4) (at 39.37 97.79 0)
       (effects (font (size 1.27 1.27)) hide)
     )
@@
     (pin "T")
   )
-  (symbol (lib_id "Connector:AudioJack4") (at 62.23 63.5 180) (unit 1)
-    (in_bom yes) (on_board yes) (fields_autoplaced)
-    (property "Reference" "J105" (id 0) (at 71.12 60.3249 0)
-      (effects (font (size 1.27 1.27)) (justify right))
-    )
-    (property "Value" "AudioJack4" (id 1) (at 71.12 62.8649 0)
-      (effects (font (size 1.27 1.27)) (justify right))
-    )
-    (property "Footprint" "Footprints:TRRS-PJ-320A" (id 2) (at 62.23 63.5 0)
+  (symbol (lib_name "AudioJack4_1") (lib_id "Connector:AudioJack4") (at 62.23 63.5 180) (unit 1)
+    (in_bom yes) (on_board yes) (fields_autoplaced)
+    (property "Reference" "J105" (id 0) (at 59.69 71.7551 0)
+      (effects (font (size 1.27 1.27)) (justify right))
+    )
+    (property "Value" "AudioJack4" (id 1) (at 59.69 69.2151 0)
+      (effects (font (size 1.27 1.27)) (justify right))
+    )
+    (property "Footprint" "Footprints:TRRS-PJ-320A" (id 2) (at 62.23 53.34 0)
       (effects (font (size 1.27 1.27)) hide)
     )
@@
       (effects (font (size 1.27 1.27)) hide)
     )
+    (property "JLCPCB" "C7519" (id 4) (at 38.1 40.64 0)
+      (effects (font (size 1.27 1.27)) hide)
+    )

Commit message: More work on MCU
Connections:
- net L_RX: no longer J105.R2, U105.1 (I/O1)
- net L_TX: no longer J105.R1, U105.3 (I/O2)
- new net L_RX_CONN: J105.R2, U105.1 (I/O1)
- new net L_TX_CONN: J105.R1, U105.3 (I/O2)
Changed lines of the file:
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@@
     (stroke (width 0) (type default) (color 0 0 0 0))
   )
-  (wire (pts (xy 49.53 52.07) (xy 57.15 52.07))
+  (wire (pts (xy 43.18 52.07) (xy 57.15 52.07))
     (stroke (width 0) (type default) (color 0 0 0 0))
   )
@@
     (stroke (width 0) (type default) (color 0 0 0 0))
   )
-  (wire (pts (xy 57.15 60.96) (xy 49.53 60.96))
+  (wire (pts (xy 57.15 60.96) (xy 43.18 60.96))
     (stroke (width 0) (type default) (color 0 0 0 0))
   )
@@
     (stroke (width 0) (type default) (color 0 0 0 0))
   )
-  (wire (pts (xy 49.53 60.96) (xy 49.53 52.07))
+  (wire (pts (xy 43.18 60.96) (xy 43.18 52.07))
     (stroke (width 0) (type default) (color 0 0 0 0))
   )
@@
     (effects (font (size 1.27 1.27)) (justify left bottom))
   )
-  (label "L_RX" (at 52.07 63.5 0)
+  (label "L_RX_CONN" (at 44.45 63.5 0)
     (effects (font (size 1.27 1.27)) (justify left bottom))
   )
-  (label "L_TX" (at 52.07 60.96 0)
+  (label "L_TX_CONN" (at 44.45 60.96 0)
     (effects (font (size 1.27 1.27)) (justify left bottom))
   )

Commit message: Left side 'done'
Connections:
- net +3.3V: no longer U105.5 (VBUS)
- net +3V3: now also U105.5 (VBUS)
Changed lines of the file:
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@@
     (effects (font (size 1.27 1.27)) (justify right))
-  )
-  (symbol (lib_id "power:+3.3V") (at 38.1 27.94 0) (unit 1)
-    (in_bom yes) (on_board yes)
-    (property "Reference" "#PWR0133" (id 0) (at 38.1 31.75 0)
-      (effects (font (size 1.27 1.27)) hide)
-    )
-    (property "Value" "+3.3V" (id 1) (at 38.1 24.13 0))
-    (property "Footprint" "" (id 2) (at 38.1 27.94 0)
-      (effects (font (size 1.27 1.27)) hide)
-    )
-    (property "Datasheet" "" (id 3) (at 38.1 27.94 0)
-      (effects (font (size 1.27 1.27)) hide)
-    )
-    (pin "1")
   )
   (symbol (lib_id "power:GND") (at 38.1 54.61 0) (unit 1)
@@
       (effects (font (size 1.27 1.27)) hide)
     )
+    (pin "1")
+  )
+  (symbol (lib_id "power:+3V3") (at 38.1 27.94 0) (unit 1)
+    (in_bom yes) (on_board yes)
+    (property "Reference" "#PWR0133" (id 0) (at 38.1 31.75 0)
+      (effects (font (size 1.27 1.27)) hide)
+    )
+    (property "Value" "+3V3" (id 1) (at 38.481 23.5458 0))
+    (property "Footprint" "" (id 2) (at 38.1 27.94 0)
+      (effects (font (size 1.27 1.27)) hide)
+    )
+    (property "Datasheet" "" (id 3) (at 38.1 27.94 0)
+      (effects (font (size 1.27 1.27)) hide)
+    )

Commit message: Right ride
Connections:
- net +3.3V is gone; now on net +3V3: U205.5 (VBUS)
- net R_RX: no longer J205.R1, U205.3 (I/O2)
- net R_TX: no longer J205.R2, U205.1 (I/O1)
- new net R_RX_CONN: J205.R1, U205.3 (I/O2)
- new net R_TX_CONN: J205.R2, U205.1 (I/O1)
Changed lines of the file:
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@@
     (stroke (width 0) (type default) (color 0 0 0 0))
   )
-  (wire (pts (xy 50.8 118.11) (xy 50.8 109.22))
+  (wire (pts (xy 44.45 118.11) (xy 44.45 109.22))
     (stroke (width 0) (type default) (color 0 0 0 0))
   )
@@
     (stroke (width 0) (type default) (color 0 0 0 0))
   )
-  (wire (pts (xy 58.42 118.11) (xy 50.8 118.11))
+  (wire (pts (xy 58.42 118.11) (xy 44.45 118.11))
     (stroke (width 0) (type default) (color 0 0 0 0))
   )
@@
     (stroke (width 0) (type default) (color 0 0 0 0))
   )
-  (wire (pts (xy 50.8 109.22) (xy 58.42 109.22))
+  (wire (pts (xy 44.45 109.22) (xy 58.42 109.22))
     (stroke (width 0) (type default) (color 0 0 0 0))
   )
@@
     (effects (font (size 2.54 2.54)) (justify left bottom))
   )
-  (label "R_TX" (at 53.34 120.65 0)
+  (label "R_TX_CONN" (at 45.72 120.65 0)
     (effects (font (size 1.27 1.27)) (justify left bottom))
   )
@@
     (effects (font (size 1.27 1.27)) (justify left bottom))
   )
-  (label "R_RX" (at 53.34 118.11 0)
+  (label "R_RX_CONN" (at 45.72 118.11 0)
     (effects (font (size 1.27 1.27)) (justify left bottom))
   )
@@
     (pin "1")
   )
+  (symbol (lib_id "power:+3V3") (at 39.37 85.09 0) (unit 1)
+    (in_bom yes) (on_board yes)
+    (property "Reference" "#PWR0140" (id 0) (at 39.37 88.9 0)
+      (effects (font (size 1.27 1.27)) hide)
+    )
+    (property "Value" "+3V3" (id 1) (at 39.751 80.6958 0))
+    (property "Footprint" "" (id 2) (at 39.37 85.09 0)
+      (effects (font (size 1.27 1.27)) hide)
+    )
+    (property "Datasheet" "" (id 3) (at 39.37 85.09 0)
+      (effects (font (size 1.27 1.27)) hide)
+    )
+    (pin "1")
+  )
   (symbol (lib_id "power:+3V3") (at 38.1 27.94 0) (unit 1)
     (in_bom yes) (on_board yes)
@@
       (effects (font (size 1.27 1.27)) hide)
     )
-    (pin "1")
-  )
-  (symbol (lib_id "power:+3.3V") (at 39.37 85.09 0) (unit 1)
-    (in_bom yes) (on_board yes) (fields_autoplaced)
-    (property "Reference" "#PWR0233" (id 0) (at 39.37 88.9 0)
-      (effects (font (size 1.27 1.27)) hide)
-    )
-    (property "Value" "+3.3V" (id 1) (at 39.37 80.01 0))
-    (property "Footprint" "" (id 2) (at 39.37 85.09 0)
-      (effects (font (size 1.27 1.27)) hide)
-    )
-    (property "Datasheet" "" (id 3) (at 39.37 85.09 0)
-      (effects (font (size 1.27 1.27)) hide)
-    )
